Commit message: updated left and right hand

File: 02-dual_proxy_motion_normal_force_robot/panda_arm_allegro.urdf (robot description, URDF)
Before this commit: robot panda, 30 links, 29 joints
Links:
- link end_effector: geometry collision sphere radius=0.035

File: 02-dual_proxy_motion_normal_force_robot/panda_arm_allegro_left.urdf (robot description, URDF)
Before this commit: robot panda, 30 links, 29 joints
Links:
- link end_effector: geometry collision sphere radius=0.035
