Commit message: Began process of stripping out unnecessary elements for basic simulation.

File: 00-ball_reorient/allegro_hand.urdf (robot description, URDF)
Before this commit: robot panda_with_allegro, 30 links, 29 joints
Links:
- removed link end_effector
- removed link link0
- removed link link1
- removed link link2
- removed link link3
- removed link link4
- removed link link5
- removed link link6
- removed link link7
Joints:
- removed joint hand_connection
- removed joint joint1
- removed joint joint2
- removed joint joint3
- removed joint joint4
- removed joint joint5
- removed joint joint6
- removed joint joint7
- removed joint joint_fixed
