Commit message: fix: partial version of hand and arm control

File: 00-ball_reorient/panda_arm_allegro.urdf (robot description, URDF)
Before this commit: robot panda_with_allegro, 30 links, 29 joints
Links:
- link link0: geometry visual mesh filename=../../../model/meshes/visual/link0.obj
- link link1: geometry visual mesh filename=../../../model/meshes/visual/link1.obj
- link link2: geometry visual mesh filename=../../../model/meshes/visual/link2.obj
- link link3: geometry visual mesh filename=../../../model/meshes/visual/link3.obj
- link link4: geometry visual mesh filename=../../../model/meshes/visual/link4.obj
- link link5: geometry visual mesh filename=../../../model/meshes/visual/link5.obj
- link link6: geometry visual mesh filename=../../../model/meshes/visual/link6.obj
- link link7: geometry visual mesh filename=../../../model/meshes/visual/link7.obj
- link link_0: geometry collision mesh filename=../../../model/allegro/link_0.0.obj; visual mesh filename=../../../model/allegro/link_0.0.obj
- link link_1: geometry collision mesh filename=../../../model/allegro/link_1.0.obj; visual mesh filename=../../../model/allegro/link_1.0.obj
- link link_10: geometry collision mesh filename=../../../model/allegro/link_2.0.obj; visual mesh filename=../../../model/allegro/link_2.0.obj
- link link_11: geometry collision mesh filename=../../../model/allegro/link_3.0.obj; visual mesh filename=../../../model/allegro/link_3.0.obj
- link link_11_tip: geometry collision sphere radius=0.012; visual mesh filename=../../../model/allegro/link_3.0_tip.obj
- link link_12: geometry collision mesh filename=../../../model/allegro/link_12.0_right.obj; visual mesh filename=../../../model/allegro/link_12.0_right.obj
- link link_13: geometry collision mesh filename=../../../model/allegro/link_13.0.obj; visual mesh filename=../../../model/allegro/link_13.0.obj
- link link_14: geometry collision mesh filename=../../../model/allegro/link_14.0.obj; visual mesh filename=../../../model/allegro/link_14.0.obj
- link link_15: geometry collision mesh filename=../../../model/allegro/link_15.0.obj; visual mesh filename=../../../model/allegro/link_15.0.obj
- link link_15_tip: geometry collision sphere radius=0.012; visual mesh filename=../../../model/allegro/link_15.0_tip.obj
- link link_2: geometry collision mesh filename=../../../model/allegro/link_2.0.obj; visual mesh filename=../../../model/allegro/link_2.0.obj
- link link_3: geometry collision mesh filename=../../../model/allegro/link_3.0.obj; visual mesh filename=../../../model/allegro/link_3.0.obj
- link link_3_tip: geometry collision sphere radius=0.012; visual mesh filename=../../../model/allegro/link_3.0_tip.obj
- link link_4: geometry collision mesh filename=../../../model/allegro/link_0.0.obj; visual mesh filename=../../../model/allegro/link_0.0.obj
- link link_5: geometry collision mesh filename=../../../model/allegro/link_1.0.obj; visual mesh filename=../../../model/allegro/link_1.0.obj
- link link_6: geometry collision mesh filename=../../../model/allegro/link_2.0.obj; visual mesh filename=../../../model/allegro/link_2.0.obj
- link link_7: geometry collision mesh filename=../../../model/allegro/link_3.0.obj; visual mesh filename=../../../model/allegro/link_3.0.obj
- link link_7_tip: geometry collision sphere radius=0.012; visual mesh filename=../../../model/allegro/link_3.0_tip.obj
- link link_8: geometry collision mesh filename=../../../model/allegro/link_0.0.obj; visual mesh filename=../../../model/allegro/link_0.0.obj
- link link_9: geometry collision mesh filename=../../../model/allegro/link_1.0.obj; visual mesh filename=../../../model/allegro/link_1.0.obj
- link palm_link: geometry collision box size=0.0407 0.1125 0.093; visual mesh filename=../../../model/allegro/base_link.obj

File: 1-panda_with_allegro/panda_arm.urdf (robot description, URDF)
Before this commit: robot panda, 8 links, 7 joints
Links:
- added link end_effector, mass 1.0; collision sphere radius=0.035
Joints:
- added joint joint_fixed: type fixed, parent link7, child end_effector, origin xyz=0 0 0.142 rpy=0 0 0
