Commit message: Working joint position controller via dynamic decoupling Minor naming update for Allegro Hand URDF

File: 0-allegro_hand_only/allegro_hand.urdf (robot description, URDF)
Before this commit: robot allegro, 21 links, 20 joints
Links:
- link link_0: geometry collision mesh filename=../../../model/allegro/link_0.0.obj; visual mesh filename=../../../model/allegro/link_0.0.obj
- link link_1: geometry collision mesh filename=../../../model/allegro/link_1.0.obj; visual mesh filename=../../../model/allegro/link_1.0.obj
- link link_10: geometry collision mesh filename=../../../model/allegro/link_2.0.obj; visual mesh filename=../../../model/allegro/link_2.0.obj
- link link_11: geometry collision mesh filename=../../../model/allegro/link_3.0.obj; visual mesh filename=../../../model/allegro/link_3.0.obj
- link link_11_tip: geometry collision sphere radius=0.012; visual mesh filename=../../../model/allegro/link_3.0_tip.obj
- link link_12: geometry collision mesh filename=../../../model/allegro/link_12.0_right.obj; visual mesh filename=../../../model/allegro/link_12.0_right.obj
- link link_13: geometry collision mesh filename=../../../model/allegro/link_13.0.obj; visual mesh filename=../../../model/allegro/link_13.0.obj
- link link_14: geometry collision mesh filename=../../../model/allegro/link_14.0.obj; visual mesh filename=../../../model/allegro/link_14.0.obj
- link link_15: geometry collision mesh filename=../../../model/allegro/link_15.0.obj; visual mesh filename=../../../model/allegro/link_15.0.obj
- link link_15_tip: geometry collision sphere radius=0.012; visual mesh filename=../../../model/allegro/link_15.0_tip.obj
- link link_2: geometry collision mesh filename=../../../model/allegro/link_2.0.obj; visual mesh filename=../../../model/allegro/link_2.0.obj
- link link_3: geometry collision mesh filename=../../../model/allegro/link_3.0.obj; visual mesh filename=../../../model/allegro/link_3.0.obj
- link link_3_tip: geometry collision sphere radius=0.012; visual mesh filename=../../../model/allegro/link_3.0_tip.obj
- link link_4: geometry collision mesh filename=../../../model/allegro/link_0.0.obj; visual mesh filename=../../../model/allegro/link_0.0.obj
- link link_5: geometry collision mesh filename=../../../model/allegro/link_1.0.obj; visual mesh filename=../../../model/allegro/link_1.0.obj
- link link_6: geometry collision mesh filename=../../../model/allegro/link_2.0.obj; visual mesh filename=../../../model/allegro/link_2.0.obj
- link link_7: geometry collision mesh filename=../../../model/allegro/link_3.0.obj; visual mesh filename=../../../model/allegro/link_3.0.obj
- link link_7_tip: geometry collision sphere radius=0.012; visual mesh filename=../../../model/allegro/link_3.0_tip.obj
- link link_8: geometry collision mesh filename=../../../model/allegro/link_0.0.obj; visual mesh filename=../../../model/allegro/link_0.0.obj
- link link_9: geometry collision mesh filename=../../../model/allegro/link_1.0.obj; visual mesh filename=../../../model/allegro/link_1.0.obj
- link palm_link: geometry collision box size=0.0407 0.1125 0.093; visual mesh filename=../../../model/allegro/base_link.obj

Commit message: Intermediate Results Commit

File: 0-allegro_hand_only/allegro_hand.urdf (robot description, URDF)
Before this commit: robot allegro, 21 links, 20 joints
Links:
- link link_0: geometry visual mesh filename=../../../model/allegro/link_0.0.obj
- link link_1: geometry visual mesh filename=../../../model/allegro/link_1.0.obj
- link link_10: geometry visual mesh filename=../../../model/allegro/link_2.0.obj
- link link_11: geometry visual mesh filename=../../../model/allegro/link_3.0.obj
- link link_11_tip: geometry visual mesh filename=../../../model/allegro/link_3.0_tip.obj
- link link_12: geometry visual mesh filename=../../../model/allegro/link_12.0_right.obj
- link link_13: geometry visual mesh filename=../../../model/allegro/link_13.0.obj
- link link_14: geometry visual mesh filename=../../../model/allegro/link_14.0.obj
- link link_15: geometry visual mesh filename=../../../model/allegro/link_15.0.obj
- link link_15_tip: geometry visual mesh filename=../../../model/allegro/link_15.0_tip.obj
- link link_2: geometry visual mesh filename=../../../model/allegro/link_2.0.obj
- link link_3: geometry visual mesh filename=../../../model/allegro/link_3.0.obj
- link link_3_tip: geometry visual mesh filename=../../../model/allegro/link_3.0_tip.obj
- link link_4: geometry visual mesh filename=../../../model/allegro/link_0.0.obj
- link link_5: geometry visual mesh filename=../../../model/allegro/link_1.0.obj
- link link_6: geometry visual mesh filename=../../../model/allegro/link_2.0.obj
- link link_7: geometry visual mesh filename=../../../model/allegro/link_3.0.obj
- link link_7_tip: geometry visual mesh filename=../../../model/allegro/link_3.0_tip.obj
- link link_8: geometry visual mesh filename=../../../model/allegro/link_0.0.obj
- link link_9: geometry visual mesh filename=../../../model/allegro/link_1.0.obj

Commit message: fix: add original urdf

File: 0-allegro_hand_only/allegro_hand.urdf (robot description, URDF)
Before this commit: robot allegro, 21 links, 20 joints
Links:
- removed link link_0
- removed link link_1
- removed link link_10
- removed link link_11
- removed link link_11_tip
- removed link link_12
- removed link link_13
- removed link link_14
- removed link link_15
- removed link link_15_tip
- removed link link_2
- removed link link_3
- removed link link_3_tip
- removed link link_4
- removed link link_5
- removed link link_6
- removed link link_7
- removed link link_7_tip
- removed link link_8
- removed link link_9
- added link link_0.0, mass 0.0119; visual mesh filename=../../../model/allegro/link_0.0.obj
- added link link_1.0, mass 0.065; visual mesh filename=../../../model/allegro/link_1.0.obj
- added link link_10.0, mass 0.0355; visual mesh filename=../../../model/allegro/link_2.0.obj
- added link link_11.0, mass 0.0096; visual mesh filename=../../../model/allegro/link_3.0.obj
- added link link_11.0_tip, mass 0.0168; visual mesh filename=../../../model/allegro/link_3.0_tip.obj
- added link link_12.0, mass 0.0176; visual mesh filename=../../../model/allegro/link_12.0_right.obj
- added link link_13.0, mass 0.0119; visual mesh filename=../../../model/allegro/link_13.0.obj
- added link link_14.0, mass 0.038; visual mesh filename=../../../model/allegro/link_14.0.obj
- added link link_15.0, mass 0.0388; visual mesh filename=../../../model/allegro/link_15.0.obj
- added link link_15.0_tip, mass 0.0168; visual mesh filename=../../../model/allegro/link_15.0_tip.obj
- added link link_2.0, mass 0.0355; visual mesh filename=../../../model/allegro/link_2.0.obj
- added link link_3.0, mass 0.0096; visual mesh filename=../../../model/allegro/link_3.0.obj
- added link link_3.0_tip, mass 0.0168; visual mesh filename=../../../model/allegro/link_3.0_tip.obj
- added link link_4.0, mass 0.0119; visual mesh filename=../../../model/allegro/link_0.0.obj
- added link link_5.0, mass 0.065; visual mesh filename=../../../model/allegro/link_1.0.obj
- added link link_6.0, mass 0.0355; visual mesh filename=../../../model/allegro/link_2.0.obj
- added link link_7.0, mass 0.0096; visual mesh filename=../../../model/allegro/link_3.0.obj
- added link link_7.0_tip, mass 0.0168; visual mesh filename=../../../model/allegro/link_3.0_tip.obj
- added link link_8.0, mass 0.0119; visual mesh filename=../../../model/allegro/link_0.0.obj
- added link link_9.0, mass 0.065; visual mesh filename=../../../model/allegro/link_1.0.obj
- link palm_link: geometry visual mesh filename=../../../model/allegro/base_link.obj
Joints:
- removed joint joint_0
- removed joint joint_1
- removed joint joint_10
- removed joint joint_11
- removed joint joint_11_tip
- removed joint joint_12
- removed joint joint_13
- removed joint joint_14
- removed joint joint_15
- removed joint joint_15_tip
- removed joint joint_2
- removed joint joint_3
- removed joint joint_3_tip
- removed joint joint_4
- removed joint joint_5
- removed joint joint_6
- removed joint joint_7
- removed joint joint_7_tip
- removed joint joint_8
- removed joint joint_9
- added joint joint_0.0: type revolute, parent palm_link, child link_0.0, origin xyz=0 0.0435 -0.001542 rpy=-0.08726646255 0 0, axis 0 0 1, limit lower=-0.47 upper=0.47 effort=15 velocity=7
- added joint joint_1.0: type revolute, parent link_0.0, child link_1.0, origin xyz=0 0 0.0164, axis 0 1 0, limit lower=-0.196 upper=1.61 effort=15 velocity=7
- added joint joint_10.0: type revolute, parent link_9.0, child link_10.0, origin xyz=0 0 0.054, axis 0 1 0, limit lower=-0.174 upper=1.709 effort=15 velocity=7
- added joint joint_11.0: type revolute, parent link_10.0, child link_11.0, origin xyz=0 0 0.0384, axis 0 1 0, limit lower=-0.227 upper=1.618 effort=15 velocity=7
- added joint joint_11.0_tip: type fixed, parent link_11.0, child link_11.0_tip, origin xyz=0 0 0.0267 rpy=0 0 0
- added joint joint_12.0: type revolute, parent palm_link, child link_12.0, origin xyz=-0.0182 0.019333 -0.045987 rpy=0 -1.65806278845 -1.5707963259, axis 1 0 0, limit lower=0.263 upper=1.396 effort=15 velocity=7
- added joint joint_13.0: type revolute, parent link_12.0, child link_13.0, origin xyz=-0.027 0.005 0.0399, axis 0 0 1, limit lower=-0.105 upper=1.163 effort=15 velocity=7
- added joint joint_14.0: type revolute, parent link_13.0, child link_14.0, origin xyz=0 0 0.0177, axis 0 1 0, limit lower=-0.189 upper=1.644 effort=15 velocity=7
- added joint joint_15.0: type revolute, parent link_14.0, child link_15.0, origin xyz=0 0 0.0514, axis 0 1 0, limit lower=-0.162 upper=1.719 effort=15 velocity=7
- added joint joint_15.0_tip: type fixed, parent link_15.0, child link_15.0_tip, origin xyz=0 0 0.0423 rpy=0 0 0
- added joint joint_2.0: type revolute, parent link_1.0, child link_2.0, origin xyz=0 0 0.054, axis 0 1 0, limit lower=-0.174 upper=1.709 effort=15 velocity=7
- added joint joint_3.0: type revolute, parent link_2.0, child link_3.0, origin xyz=0 0 0.0384, axis 0 1 0, limit lower=-0.227 upper=1.618 effort=15 velocity=7
- added joint joint_3.0_tip: type fixed, parent link_3.0, child link_3.0_tip, origin xyz=0 0 0.0267 rpy=0 0 0
- added joint joint_4.0: type revolute, parent palm_link, child link_4.0, origin xyz=0 0 0.0007 rpy=0.0 0 0, axis 0 0 1, limit lower=-0.47 upper=0.47 effort=15 velocity=7
- added joint joint_5.0: type revolute, parent link_4.0, child link_5.0, origin xyz=0 0 0.0164, axis 0 1 0, limit lower=-0.196 upper=1.61 effort=15 velocity=7
- added joint joint_6.0: type revolute, parent link_5.0, child link_6.0, origin xyz=0 0 0.054, axis 0 1 0, limit lower=-0.174 upper=1.709 effort=15 velocity=7
- added joint joint_7.0: type revolute, parent link_6.0, child link_7.0, origin xyz=0 0 0.0384, axis 0 1 0, limit lower=-0.227 upper=1.618 effort=15 velocity=7
- added joint joint_7.0_tip: type fixed, parent link_7.0, child link_7.0_tip, origin xyz=0 0 0.0267 rpy=0 0 0
- added joint joint_8.0: type revolute, parent palm_link, child link_8.0, origin xyz=0 -0.0435 -0.001542 rpy=0.08726646255 0 0, axis 0 0 1, limit lower=-0.47 upper=0.47 effort=15 velocity=7
- added joint joint_9.0: type revolute, parent link_8.0, child link_9.0, origin xyz=0 0 0.0164, axis 0 1 0, limit lower=-0.196 upper=1.61 effort=15 velocity=7

Commit message: fix: urdf and posture

File: 0-allegro_hand_only/allegro_hand.urdf (robot description, URDF)
Before this commit: robot allegro, 21 links, 20 joints
Joints:
- joint joint_12.0: axis 1 0 0 -> -1 0 0
